Commit message: Add collision meshes
Add collision meshes for some links.
Maybe some of them too high-poly

File: xacro/arm.xacro (robot description, xacro)
@@ -10,5 +10,5 @@
 		<xacro:left_right side="${side}"/>
 		<link name="shoulder_fork_${side}">
-	 		<xacro:meshes file="shoulder_fork_${side}"/>
+	 		<xacro:meshes file="shoulder_fork_${side}" collision="True"/>
 	 		<inertial>
 	 			<!-- should be 0.04, but -0.04 fits -->
@@ -21,5 +21,5 @@
 	 	</link>
 	 	<link name="shoulder_${side}">
-	 		<xacro:meshes file="shoulder_${side}"/>
+	 		<xacro:meshes file="shoulder_${side}" collision="True"/>
 	 		<inertial>
 	 			<origin xyz="0 0 -0.05" rpy="0 0 0"/>

File: xacro/head.xacro (robot description, xacro)
@@ -40,5 +40,5 @@
 	 	</link>
 	 	<link name="head">
-	 		<xacro:meshes file="head"/>
+	 		<xacro:meshes file="head" collision="True"/>
 	 		<inertial>
 	 			<origin xyz="0 0.04 0.06" rpy="0 0 0"/>

File: xacro/leg.xacro (robot description, xacro)
@@ -11,5 +11,5 @@
 		<!-- Links -->
 		<link name="hip_fork_${side}">
-	 		<xacro:meshes file="hip_fork_${side}"/>
+	 		<xacro:meshes file="hip_fork_${side}" collision="True"/>
 	 		<inertial>
 	 			<origin xyz="0 -0.02 0.07" rpy="0 0 0"/>
@@ -31,5 +31,5 @@
 	 	</link>
 	 	<link name="hip_${side}">
-	 		<xacro:meshes file="hip_${side}"/>
+	 		<xacro:meshes file="hip_${side}" collision="True"/>
 	 		<inertial>
 	 			<origin xyz="0 0.01 -0.14" rpy="0 0 0"/>
@@ -41,5 +41,5 @@
 	 	</link>
 	 	<link name="shin_${side}">
-	 		<xacro:meshes file="shin_${side}"/>
+	 		<xacro:meshes file="shin_${side}" collision="True"/>
 	 		<inertial>
 	 			<origin xyz="${0.01 * x_sign} 0 -0.11" rpy="0 0 0"/>
@@ -61,5 +61,5 @@
 	 	</link>
 	 	<link name="foot_${side}">
-	 		<xacro:meshes file="foot_${side}"/>
+	 		<xacro:meshes file="foot_${side}" collision="True"/>
 	 		<inertial>
 	 			<origin xyz="0 0.03 -0.06" rpy="0 0 0"/>

File: xacro/meshes.xacro (robot description, xacro)
@@ -2,5 +2,5 @@
 <!-- Create visual and collision with given mesh -->
 <robot xmlns:xacro="http://www.ros.org/wiki/xacro">
-	<xacro:macro name="meshes" params="file xyz:='0 0 0' rpy:='0 0 0'">
+	<xacro:macro name="meshes" params="file xyz:='0 0 0' rpy:='0 0 0' collision='False'">
 		<visual>
  			<origin xyz="${xyz}" rpy="${rpy}"/>
@@ -12,4 +12,12 @@
      		</material>
 	 	</visual>
+	 	<xacro:if value="${collision}">
+	 		<collision>
+	 			<origin xyz="${xyz}" rpy="${rpy}"/>
+	 			<geometry>
+ 					<mesh filename="package://ar600_description/meshes/collision/${file}.stl"/>
+ 				</geometry>
+	 		</collision>
+	 	</xacro:if>
 	</xacro:macro>
 </robot>

File: xacro/pelvis.xacro (robot description, xacro)
@@ -10,5 +10,5 @@
 		<link name="base_link">
 			<!-- this shift is WTF and hack -->
-	 		<xacro:meshes file="pelvis" xyz="0 0.0276 0"/>
+	 		<xacro:meshes file="pelvis" xyz="0 0.0276 0" collision="True"/>
 	 		<inertial>
 	 			<!-- z origin is incorrect -->
@@ -19,10 +19,4 @@
       				     izz="1.0"/>
     		</inertial>
-    		<collision>
-    			<origin xyz="0 0 0.5" rpy="0 0 0"/>
-				<geometry>
-					<box size="0.5 0.5 0.5"/>
-				</geometry>
-			</collision>
 	 	</link>
  	</xacro:macro>

File: xacro/torso.xacro (robot description, xacro)
@@ -3,5 +3,5 @@
 	<xacro:macro name="torso" params="parent">
 		<link name="torso">
-	 		<xacro:meshes file="torso"/>
+	 		<xacro:meshes file="torso" collision="True"/>
 	 		<inertial>
 	 			<!-- origin is incorrect -->

Commit message: Physical parameters fixes  - Fix CoMs positions  - Add intertia tensors

File: xacro/arm.xacro (robot description, xacro)
@@ -13,9 +13,9 @@
 	 		<inertial>
 	 			<!-- should be 0.04, but -0.04 fits -->
-	 			<origin xyz="${-0.04 * x_sign} -0.01 0" rpy="0 0 0"/>
+	 			<origin xyz="${-0.01 * x_sign} -0.04 0.00" rpy="0 0 0"/>
       			<mass value="1.362"/>
-      			<inertia ixx="1.0" ixy="1.0" ixz="1.0"
-      				     iyy="1.0" iyz="1.0"
-      				     izz="1.0"/>
+      			<inertia ixx="0.001569" ixy="-0.000014" ixz="0.000068"
+      				                    iyy="0.001358"  iyz="-0.000058"
+      				                                    izz="0.002036"/>
     		</inertial>
 	 	</link>
@@ -23,9 +23,9 @@
 	 		<xacro:meshes file="shoulder_${side}" collision="True"/>
 	 		<inertial>
-	 			<origin xyz="0 0 -0.05" rpy="0 0 0"/>
+	 			<origin xyz="0.00 0.00 -0.05" rpy="0 0 0"/>
       			<mass value="1.558"/>
-      			<inertia ixx="1.0" ixy="1.0" ixz="1.0"
-      				     iyy="1.0" iyz="1.0"
-      				     izz="1.0"/>
+      			<inertia ixx="0.002694" ixy="0.000468" ixz="-0.000004"
+      				                    iyy="0.001001" iyz="-0.000005"
+      				                                   izz="0.002996"/>
     		</inertial>
 	 	</link>

File: xacro/head.xacro (robot description, xacro)
@@ -11,9 +11,9 @@
 	 		<xacro:meshes file="neck"/>
 	 		<inertial>
-	 			<origin xyz="0 -0.02 0.02" rpy="0 0 0"/>
+	 			<origin xyz="-0.02 0.00 0.02" rpy="0 0 0"/>
       			<mass value="0.633"/>
-      			<inertia ixx="1.0" ixy="1.0" ixz="1.0"
-      				     iyy="1.0" iyz="1.0"
-      				     izz="1.0"/>
+      			<inertia ixx="0.000884" ixy="0.000001" ixz="-0.000246"
+      				                    iyy="0.000982" iyz="0.000500"
+      				                                   izz="0.000627"/>
     		</inertial>
 	 	</link>
@@ -24,7 +24,7 @@
 	 			<origin xyz="0.01 -0.01 -0.02" rpy="0 0 0"/>
       			<mass value="0.444"/>
-      			<inertia ixx="1.0" ixy="1.0" ixz="1.0"
-      				     iyy="1.0" iyz="1.0"
-      				     izz="1.0"/>
+      			<inertia ixx="0.000285" ixy="-0.000016" ixz="0.000073"
+      				                    iyy="0.000401"  iyz="-0.000021"
+      				                                    izz="0.000238"/>
     		</inertial>
 	 	</link>
@@ -32,9 +32,9 @@
 	 		<xacro:meshes file="neck_cross"/>
 	 		<inertial>
-	 			<origin xyz="-0.01 0.01 0" rpy="0 0 0"/>
+	 			<origin xyz="0.01 0.01 0" rpy="0 0 0"/>
       			<mass value="0.320"/>
-      			<inertia ixx="1.0" ixy="1.0" ixz="1.0"
-      				     iyy="1.0" iyz="1.0"
-      				     izz="1.0"/>
+      			<inertia ixx="0.000054" ixy="-0.000002" ixz="0.000000"
+      				                    iyy="0.000054"  iyz="0.000000"
+      				                                    izz="0.000092"/>
     		</inertial>
 	 	</link>
@@ -42,9 +42,9 @@
 	 		<xacro:meshes file="head" collision="True"/>
 	 		<inertial>
-	 			<origin xyz="0 0.04 0.06" rpy="0 0 0"/>
+	 			<origin xyz="0.04 0.00 0.06" rpy="0 0 0"/>
       			<mass value="1.258"/>
-      			<inertia ixx="1.0" ixy="1.0" ixz="1.0"
-      				     iyy="1.0" iyz="1.0"
-      				     izz="1.0"/>
+      			<inertia ixx="0.005118" ixy="-0.000058" ixz="-0.000120"
+      				                    iyy="0.005112"  iyz="-0.000172"
+      				                                    izz="0.005643"/>
     		</inertial>
 	 	</link>

File: xacro/leg.xacro (robot description, xacro)
@@ -3,7 +3,7 @@
 	<!--
 		Solid Works conversion
-		x <- -x
-		y <-  z
-		z <-  y
+		x <- z
+		y <- x
+		z <- y
 	-->
 	<xacro:macro name="leg" params="parent side">
@@ -13,9 +13,9 @@
 	 		<xacro:meshes file="hip_fork_${side}" collision="True"/>
 	 		<inertial>
-	 			<origin xyz="0 -0.02 0.07" rpy="0 0 0"/>
+	 			<origin xyz="${-0.02 * x_sign} 0 0.07" rpy="0 0 0"/>
       			<mass value="3.170"/>
-      			<inertia ixx="1.0" ixy="1.0" ixz="1.0"
-      				     iyy="1.0" iyz="1.0"
-      				     izz="1.0"/>
+      			<inertia ixx="0.009316" ixy="-0.000234" ixz="0.002895"
+      				                    iyy="0.012979"  iyz="0.000000"
+      				                                    izz="0.006561"/>
     		</inertial>
 	 	</link>
@@ -23,9 +23,9 @@
 	 		<xacro:meshes file="hip_cross_${side}"/>
 	 		<inertial>
-	 			<origin xyz="${-0.01 * x_sign} -0.03 0" rpy="0 0 0"/>
+	 			<origin xyz="${-0.03 * x_sign} 0.01 0.00" rpy="0 0 0"/>
       			<mass value="1.799"/>
-      			<inertia ixx="1.0" ixy="1.0" ixz="1.0"
-      				     iyy="1.0" iyz="1.0"
-      				     izz="1.0"/>
+      			<inertia ixx="0.001498" ixy="0.000126" ixz="0.000001"
+      				                    iyy="0.001990" iyz="-0.000016"
+      				                                   izz="0.002404"/>
     		</inertial>
 	 	</link>
@@ -33,9 +33,9 @@
 	 		<xacro:meshes file="hip_${side}" collision="True"/>
 	 		<inertial>
-	 			<origin xyz="0 0.01 -0.14" rpy="0 0 0"/>
+	 			<origin xyz="${0.01 * x_sign} 0.00 -0.14" rpy="0 0 0"/>
       			<mass value="6.779"/>
-      			<inertia ixx="1.0" ixy="1.0" ixz="1.0"
-      				     iyy="1.0" iyz="1.0"
-      				     izz="1.0"/>
+      			<inertia ixx="0.037615" ixy="0.000139" ixz="-0.000896"
+      				                    iyy="0.031299" iyz="-0.000182"
+      				                                   izz="0.012270"/>
     		</inertial>
 	 	</link>
@@ -43,9 +43,9 @@
 	 		<xacro:meshes file="shin_${side}" collision="True"/>
 	 		<inertial>
-	 			<origin xyz="${0.01 * x_sign} 0 -0.11" rpy="0 0 0"/>
+	 			<origin xyz="0.00 0.01 -0.11" rpy="0 0 0"/>
       			<mass value="1"/>
-      			<inertia ixx="1.0" ixy="1.0" ixz="1.0"
-      				     iyy="1.0" iyz="1.0"
-      				     izz="1.0"/>
+      			<inertia ixx="0.028848" ixy="0.000053" ixz="-0.000056"
+      				                    iyy="0.026849" iyz="0.001709"
+      				                                   izz="0.005196"/>
     		</inertial>
 	 	</link>
@@ -53,9 +53,9 @@
 	 		<xacro:meshes file="ankle_${side}"/>
 	 		<inertial>
-	 			<origin xyz="${-0.01 * x_sign} -0.02 0" rpy="0 0 0"/>
+	 			<origin xyz="${-0.02 * x_sign} 0.01 0.00" rpy="0 0 0"/>
       			<mass value="1"/>
-      			<inertia ixx="1.0" ixy="1.0" ixz="1.0"
-      				     iyy="1.0" iyz="1.0"
-      				     izz="1.0"/>
+      			<inertia ixx="0.000424" ixy="-0.000001" ixz="-0.000001"
+      				                    iyy="0.000603"  iyz="0.000001"
+      				                                    izz="0.000898"/>
     		</inertial>
 	 	</link>
@@ -63,9 +63,9 @@
 	 		<xacro:meshes file="foot_${side}" collision="True"/>
 	 		<inertial>
-	 			<origin xyz="0 0.03 -0.06" rpy="0 0 0"/>
+	 			<origin xyz="${0.03 * x_sign} 0.00 -0.06" rpy="0 0 0"/>
       			<mass value="1"/>
-      			<inertia ixx="1.0" ixy="1.0" ixz="1.0"
-      				     iyy="1.0" iyz="1.0"
-      				     izz="1.0"/>
+      			<inertia ixx="0.006101" ixy="-0.000307" ixz="-0.001261"
+      				                    iyy="0.012336"  iyz="0.000060"
+      				                                    izz="0.013546"/>
     		</inertial>
 	 	</link>

File: xacro/pelvis.xacro (robot description, xacro)
@@ -3,7 +3,7 @@
 	<!--
 		Solid Works conversion
-		x <- -x
-		y <-  z
-		z <-  y
+		x <- z
+		y <- x
+		z <- z
 	-->
 	<xacro:macro name="pelvis">
@@ -15,7 +15,7 @@
 	 			<origin xyz="0 0 0.15" rpy="0 0 0"/>
       			<mass value="5.045"/>
-      			<inertia ixx="1.0" ixy="1.0" ixz="1.0"
-      				     iyy="1.0" iyz="1.0"
-      				     izz="1.0"/>
+      			<inertia ixx="0.031053" ixy="0.000014" ixz="-0.000227"
+      				                    iyy="0.012429" iyz="-0.000016"
+      				                                   izz="0.032811"/>
     		</inertial>
 	 	</link>

File: xacro/torso.xacro (robot description, xacro)
@@ -6,9 +6,9 @@
 	 		<inertial>
 	 			<!-- origin is incorrect -->
-	 			<origin xyz="0 0 -0.16" rpy="0 0 0"/>
+	 			<origin xyz="0 0 -0.09" rpy="0 0 0"/>
       			<mass value="29.642"/>
-      			<inertia ixx="1.0" ixy="1.0" ixz="1.0"
-      				     iyy="1.0" iyz="1.0"
-      				     izz="1.0"/>
+      			<inertia ixx="0.118418" ixy="-0.000174" ixz="0.001227"
+      				                    iyy="0.091310"  iyz="-0.000488"
+      				                                    izz="0.061124"/>
     		</inertial>
 	 	</link>

Commit message: Made reverse for joints

File: xacro/arm.xacro (robot description, xacro)
@@ -46,5 +46,5 @@
 	 		<child link="shoulder_${side}"/>
 	 		<origin xyz="0 0 0" rpy="0 0 0"/>
-	 		<axis xyz="0 1 0"/>
+	 		<axis xyz="0 ${-x_sign} 0"/>
 	 		<xacro:lr_limit side="${side}" lower="0" upper="${105*d2r}" effort="10" velocity="10"/>
 	 	</joint>

File: xacro/leg.xacro (robot description, xacro)
@@ -76,5 +76,5 @@
 	 		<child link="hip_fork_${side}"/>
 	 		<origin xyz="${0.088 * x_sign} 0.0276 0" rpy="0 0 0"/>
-	 		<axis xyz="0 0 1"/>
+	 		<axis xyz="0 0 ${-x_sign}"/>
 	 		<limit lower="${-20*d2r}" upper="${20*d2r}" effort="10" velocity="10"/>
 	 	</joint>
@@ -85,5 +85,5 @@
 	 		<child link="hip_cross_${side}"/>
 	 		<origin xyz="0 0 0" rpy="0 0 0"/>
-	 		<axis xyz="0 1 0"/>
+	 		<axis xyz="0 ${-x_sign} 0"/>
 	 		<xacro:lr_limit side="${side}" lower="${-11*d2r}" upper="${20*d2r}" effort="10" velocity="10"/>
 	 	</joint>
@@ -121,5 +121,5 @@
 	 		<child link="foot_${side}"/>
 	 		<origin xyz="0 0 0" rpy="0 0 0"/>
-	 		<axis xyz="0 1 0"/>
+	 		<axis xyz="0 ${-x_sign} 0"/>
 	 		<xacro:lr_limit side="${side}" lower="${-20*d2r}" upper="${11*d2r}" effort="10" velocity="10"/>
 	 	</joint>
