Commit message: Add meshes for legs  * fix some positions  * add meshes  * add interial params (origin, mass, without intertial matrix),    some of CoM origins look like incorrect

File: xacro/ar600.xacro (robot description, xacro)
@@ -4,8 +4,14 @@
 	<xacro:property name="M_PI" value="3.14159"/>
 	<xacro:include filename="wtf.xacro"/>
+	<xacro:include filename="meshes.xacro"/>
+	<xacro:include filename="left_right.xacro"/>
 	<xacro:include filename="pelvis.xacro"/>
 	<xacro:include filename="leg.xacro"/>
+	<xacro:include filename="torso.xacro"/>
+	<xacro:include filename="arm.xacro"/>
 	<xacro:pelvis/>
 	<xacro:leg parent="base_link" side="left"/>
 	<xacro:leg parent="base_link" side="right"/>
+	<xacro:torso parent="base_link"/>
+	<xacro:arm parent="torso" side="left"/>
 </robot>

File: xacro/leg.xacro (robot description, xacro)
@@ -1,28 +1,60 @@
 <?xml version="1.0"?>
-<robot xmlns:xacro="http://www.ros.org/wiki/xacro" name="ar600">
+<robot xmlns:xacro="http://www.ros.org/wiki/xacro">
+	<!--
+		Solid Works conversion
+		x <- -x
+		y <-  z
+		z <-  y
+	-->
 	<xacro:macro name="leg" params="parent side">
-		<xacro:if value="${side == 'left'}">
-  			<xacro:property name="x_shift" value="-0.088" />
-		</xacro:if>
-		<xacro:if value="${side == 'right'}">
-  			<xacro:property name="x_shift" value="0.088" />
-		</xacro:if>
+		<xacro:left_right side="${side}"/>
+		<!-- Links -->
 		<link name="hip_fork_${side}">
-	 		<xacro:wtf/>
+	 		<xacro:meshes file="hip_fork_${side}"/>
+	 		<inertial>
+	 			<origin xyz="0 -0.02 0.07" rpy="0 0 0"/>
+      			<mass value="3.170"/>
+      			<inertia ixx="0.0" ixy="0.0" ixz="0.0" iyy="0.0" iyz="0.0" izz="0.0"/>
+    		</inertial>
 	 	</link>
 	 	<link name="hip_cross_${side}">
-	 		<xacro:wtf/>
+	 		<xacro:meshes file="hip_cross_${side}"/>
+	 		<inertial>
+	 			<origin xyz="${-0.01 * x_sign} -0.03 0" rpy="0 0 0"/>
+      			<mass value="1.799"/>
+      			<inertia ixx="0.0" ixy="0.0" ixz="0.0" iyy="0.0" iyz="0.0" izz="0.0"/>
+    		</inertial>
 	 	</link>
 	 	<link name="hip_${side}">
-	 		<xacro:wtf/>
+	 		<xacro:meshes file="hip_${side}"/>
+	 		<inertial>
+	 			<origin xyz="0 0.01 -0.14" rpy="0 0 0"/>
+      			<mass value="6.779"/>
+      			<inertia ixx="0.0" ixy="0.0" ixz="0.0" iyy="0.0" iyz="0.0" izz="0.0"/>
+    		</inertial>
 	 	</link>
 	 	<link name="shin_${side}">
-	 		<xacro:wtf/>
+	 		<xacro:meshes file="shin_${side}"/>
+	 		<inertial>
+	 			<origin xyz="${0.01 * x_sign} 0 -0.11" rpy="0 0 0"/>
+      			<mass value="1"/>
+      			<inertia ixx="0.0" ixy="0.0" ixz="0.0" iyy="0.0" iyz="0.0" izz="0.0"/>
+    		</inertial>
 	 	</link>
 	 	<link name="ankle_${side}">
-	 		<xacro:wtf/>
+	 		<xacro:meshes file="ankle_${side}"/>
+	 		<inertial>
+	 			<origin xyz="${-0.01 * x_sign} -0.02 0" rpy="0 0 0"/>
+      			<mass value="1"/>
+      			<inertia ixx="0.0" ixy="0.0" ixz="0.0" iyy="0.0" iyz="0.0" izz="0.0"/>
+    		</inertial>
 	 	</link>
 	 	<link name="foot_${side}">
-	 		<xacro:wtf/>
+	 		<xacro:meshes file="foot_${side}"/>
+	 		<inertial>
+	 			<origin xyz="0 0.03 -0.06" rpy="0 0 0"/>
+      			<mass value="1"/>
+      			<inertia ixx="0.0" ixy="0.0" ixz="0.0" iyy="0.0" iyz="0.0" izz="0.0"/>
+    		</inertial>
 	 	</link>
 	 	<!-- hip z rotate (vertical)-->
@@ -32,5 +64,5 @@
 	 		<child link="hip_fork_${side}"/>
 	 		<!-- z unknown -->
-	 		<origin xyz="${x_shift} 0.0276 0" rpy="0 0 0"/>
+	 		<origin xyz="${0.088 * x_sign} 0.0276 0" rpy="0 0 0"/>
 	 		<axis xyz="0 0 1"/>
 	 		<limit lower="${-20*d2r}" upper="${20*d2r}" effort="10" velocity="10"/>
@@ -41,6 +73,6 @@
 	 		<parent link="hip_fork_${side}"/>
 	 		<child link="hip_cross_${side}"/>
-	 		<!-- unknown -->
-	 		<origin xyz="0 0 -0.25" rpy="0 0 0"/>
+	 		<!-- unknown z-->
+	 		<origin xyz="0 0 0" rpy="0 0 0"/>
 	 		<axis xyz="0 1 0"/>
 	 		<limit lower="${-11*d2r}" upper="${20*d2r}" effort="10" velocity="10"/>

File: xacro/pelvis.xacro (robot description, xacro)
@@ -1,12 +1,26 @@
 <?xml version="1.0"?>
-<robot xmlns:xacro="http://www.ros.org/wiki/xacro" name="ar600">
+<robot xmlns:xacro="http://www.ros.org/wiki/xacro">
+	<!--
+		Solid Works conversion
+		x <- -x
+		y <-  z
+		z <-  y
+	-->
 	<xacro:macro name="pelvis">
 		<link name="base_link">
-	 		<xacro:wtf/>
+			<!-- this shift is WTF and hack -->
+	 		<xacro:meshes file="pelvis" xyz="0 0.0276 0"/>
 	 		<inertial>
-	 			<origin xyz="0 0.05 0" rpy="0 0 0"/>
+	 			<!-- z origin is incorrect -->
+	 			<origin xyz="0 0 0.05" rpy="0 0 0"/>
       			<mass value="5.045"/>
       			<inertia ixx="0.0" ixy="0.0" ixz="0.0" iyy="0.0" iyz="0.0" izz="0.0"/>
     		</inertial>
+    		<collision>
+    			<origin xyz="0 0 0.5" rpy="0 0 0"/>
+				<geometry>
+					<box size="0.5 0.5 0.5"/>
+				</geometry>
+			</collision>
 	 	</link>
  	</xacro:macro>

Commit message: Create arms with meshes

File: xacro/ar600.xacro (robot description, xacro)
@@ -10,4 +10,5 @@
 	<xacro:include filename="torso.xacro"/>
 	<xacro:include filename="arm.xacro"/>
+	<xacro:include filename="head.xacro"/>
 	<xacro:pelvis/>
 	<xacro:leg parent="base_link" side="left"/>
@@ -15,3 +16,5 @@
 	<xacro:torso parent="base_link"/>
 	<xacro:arm parent="torso" side="left"/>
+	<xacro:arm parent="torso" side="right"/>
+	<xacro:head parent="torso"/>
 </robot>

File: xacro/arm.xacro (robot description, xacro)
@@ -11,4 +11,18 @@
 		<link name="shoulder_fork_${side}">
 	 		<xacro:meshes file="shoulder_fork_${side}"/>
+	 		<inertial>
+	 			<!-- should be 0.04, but -0.04 fits -->
+	 			<origin xyz="${-0.04 * x_sign} -0.01 0" rpy="0 0 0"/>
+      			<mass value="1.362"/>
+      			<inertia ixx="0.0" ixy="0.0" ixz="0.0" iyy="0.0" iyz="0.0" izz="0.0"/>
+    		</inertial>
+	 	</link>
+	 	<link name="shoulder_${side}">
+	 		<xacro:meshes file="shoulder_${side}"/>
+	 		<inertial>
+	 			<origin xyz="0 0 -0.05" rpy="0 0 0"/>
+      			<mass value="1.558"/>
+      			<inertia ixx="0.0" ixy="0.0" ixz="0.0" iyy="0.0" iyz="0.0" izz="0.0"/>
+    		</inertial>
 	 	</link>
 	 	<joint name="shoulder_f_joint_${side}"
@@ -16,8 +30,16 @@
 	 		<parent link="${parent}"/>
 	 		<child link="shoulder_fork_${side}"/>
-	 		<!-- z unknown -->
-	 		<origin xyz="${1 * x_sign} 0.0276 0" rpy="0 0 0"/>
-	 		<axis xyz="0 0 1"/>
-	 		<limit lower="${-20*d2r}" upper="${20*d2r}" effort="10" velocity="10"/>
+	 		<!-- incorrect -->
+	 		<origin xyz="${0.197 * cos(10 * d2r) * x_sign} ${0.197 * sin(10 * d2r)} 0" rpy="0 0 ${10 * d2r * x_sign}"/>
+	 		<axis xyz="1 0 0"/>
+	 		<limit lower="${-15*d2r}" upper="${90*d2r}" effort="10" velocity="10"/>
+	 	</joint>
+	 	<joint name="shoulder_s_joint_${side}"
+	 		   type="revolute">
+	 		<parent link="shoulder_fork_${side}"/>
+	 		<child link="shoulder_${side}"/>
+	 		<origin xyz="0 0 0" rpy="0 0 0"/>
+	 		<axis xyz="0 1 0"/>
+	 		<limit lower="0" upper="${105*d2r}" effort="10" velocity="10"/>
 	 	</joint>
 	</xacro:macro>

File: xacro/leg.xacro (robot description, xacro)
@@ -63,5 +63,4 @@
 	 		<parent link="${parent}"/>
 	 		<child link="hip_fork_${side}"/>
-	 		<!-- z unknown -->
 	 		<origin xyz="${0.088 * x_sign} 0.0276 0" rpy="0 0 0"/>
 	 		<axis xyz="0 0 1"/>
@@ -73,5 +72,4 @@
 	 		<parent link="hip_fork_${side}"/>
 	 		<child link="hip_cross_${side}"/>
-	 		<!-- unknown z-->
 	 		<origin xyz="0 0 0" rpy="0 0 0"/>
 	 		<axis xyz="0 1 0"/>

Commit message: Small fixes  - move pelvis and torso CoMs  - write inertia as triangle matrix

File: xacro/ar600.xacro (robot description, xacro)
@@ -3,5 +3,4 @@
 	<xacro:property name="d2r" value="0.01745329251994329577"/>
 	<xacro:property name="M_PI" value="3.14159"/>
-	<xacro:include filename="wtf.xacro"/>
 	<xacro:include filename="meshes.xacro"/>
 	<xacro:include filename="left_right.xacro"/>
@@ -17,4 +16,4 @@
 	<xacro:arm parent="torso" side="left"/>
 	<xacro:arm parent="torso" side="right"/>
-	<xacro:head parent="torso"/>
+	<!--<xacro:head parent="torso"/>-->
 </robot>

File: xacro/arm.xacro (robot description, xacro)
@@ -15,5 +15,7 @@
 	 			<origin xyz="${-0.04 * x_sign} -0.01 0" rpy="0 0 0"/>
       			<mass value="1.362"/>
-      			<inertia ixx="0.0" ixy="0.0" ixz="0.0" iyy="0.0" iyz="0.0" izz="0.0"/>
+      			<inertia ixx="1.0" ixy="1.0" ixz="1.0"
+      				     iyy="1.0" iyz="1.0"
+      				     izz="1.0"/>
     		</inertial>
 	 	</link>
@@ -23,5 +25,7 @@
 	 			<origin xyz="0 0 -0.05" rpy="0 0 0"/>
       			<mass value="1.558"/>
-      			<inertia ixx="0.0" ixy="0.0" ixz="0.0" iyy="0.0" iyz="0.0" izz="0.0"/>
+      			<inertia ixx="1.0" ixy="1.0" ixz="1.0"
+      				     iyy="1.0" iyz="1.0"
+      				     izz="1.0"/>
     		</inertial>
 	 	</link>

File: xacro/leg.xacro (robot description, xacro)
@@ -15,5 +15,7 @@
 	 			<origin xyz="0 -0.02 0.07" rpy="0 0 0"/>
       			<mass value="3.170"/>
-      			<inertia ixx="0.0" ixy="0.0" ixz="0.0" iyy="0.0" iyz="0.0" izz="0.0"/>
+      			<inertia ixx="1.0" ixy="1.0" ixz="1.0"
+      				     iyy="1.0" iyz="1.0"
+      				     izz="1.0"/>
     		</inertial>
 	 	</link>
@@ -23,5 +25,7 @@
 	 			<origin xyz="${-0.01 * x_sign} -0.03 0" rpy="0 0 0"/>
       			<mass value="1.799"/>
-      			<inertia ixx="0.0" ixy="0.0" ixz="0.0" iyy="0.0" iyz="0.0" izz="0.0"/>
+      			<inertia ixx="1.0" ixy="1.0" ixz="1.0"
+      				     iyy="1.0" iyz="1.0"
+      				     izz="1.0"/>
     		</inertial>
 	 	</link>
@@ -31,5 +35,7 @@
 	 			<origin xyz="0 0.01 -0.14" rpy="0 0 0"/>
       			<mass value="6.779"/>
-      			<inertia ixx="0.0" ixy="0.0" ixz="0.0" iyy="0.0" iyz="0.0" izz="0.0"/>
+      			<inertia ixx="1.0" ixy="1.0" ixz="1.0"
+      				     iyy="1.0" iyz="1.0"
+      				     izz="1.0"/>
     		</inertial>
 	 	</link>
@@ -39,5 +45,7 @@
 	 			<origin xyz="${0.01 * x_sign} 0 -0.11" rpy="0 0 0"/>
       			<mass value="1"/>
-      			<inertia ixx="0.0" ixy="0.0" ixz="0.0" iyy="0.0" iyz="0.0" izz="0.0"/>
+      			<inertia ixx="1.0" ixy="1.0" ixz="1.0"
+      				     iyy="1.0" iyz="1.0"
+      				     izz="1.0"/>
     		</inertial>
 	 	</link>
@@ -47,5 +55,7 @@
 	 			<origin xyz="${-0.01 * x_sign} -0.02 0" rpy="0 0 0"/>
       			<mass value="1"/>
-      			<inertia ixx="0.0" ixy="0.0" ixz="0.0" iyy="0.0" iyz="0.0" izz="0.0"/>
+      			<inertia ixx="1.0" ixy="1.0" ixz="1.0"
+      				     iyy="1.0" iyz="1.0"
+      				     izz="1.0"/>
     		</inertial>
 	 	</link>
@@ -55,5 +65,7 @@
 	 			<origin xyz="0 0.03 -0.06" rpy="0 0 0"/>
       			<mass value="1"/>
-      			<inertia ixx="0.0" ixy="0.0" ixz="0.0" iyy="0.0" iyz="0.0" izz="0.0"/>
+      			<inertia ixx="1.0" ixy="1.0" ixz="1.0"
+      				     iyy="1.0" iyz="1.0"
+      				     izz="1.0"/>
     		</inertial>
 	 	</link>

File: xacro/pelvis.xacro (robot description, xacro)
@@ -13,7 +13,9 @@
 	 		<inertial>
 	 			<!-- z origin is incorrect -->
-	 			<origin xyz="0 0 0.05" rpy="0 0 0"/>
+	 			<origin xyz="0 0 0.15" rpy="0 0 0"/>
       			<mass value="5.045"/>
-      			<inertia ixx="0.0" ixy="0.0" ixz="0.0" iyy="0.0" iyz="0.0" izz="0.0"/>
+      			<inertia ixx="1.0" ixy="1.0" ixz="1.0"
+      				     iyy="1.0" iyz="1.0"
+      				     izz="1.0"/>
     		</inertial>
     		<collision>

File: xacro/torso.xacro (robot description, xacro)
@@ -5,8 +5,10 @@
 	 		<xacro:meshes file="torso"/>
 	 		<inertial>
-	 			<!-- z origin is incorrect -->
-	 			<origin xyz="0 -0.05 0.16" rpy="0 0 0"/>
+	 			<!-- origin is incorrect -->
+	 			<origin xyz="0 0 -0.16" rpy="0 0 0"/>
       			<mass value="29.642"/>
-      			<inertia ixx="0.0" ixy="0.0" ixz="0.0" iyy="0.0" iyz="0.0" izz="0.0"/>
+      			<inertia ixx="1.0" ixy="1.0" ixz="1.0"
+      				     iyy="1.0" iyz="1.0"
+      				     izz="1.0"/>
     		</inertial>
 	 	</link>

Commit message: Add head and fix limits  - Add neck and head with CoMs  - Fix side-joints (y-axis) limits    This limits for mirrored parts (leg, arms) weren't mirrored.    Add macro to mirror revolute joint limits based on side

File: xacro/ar600.xacro (robot description, xacro)
@@ -5,4 +5,5 @@
 	<xacro:include filename="meshes.xacro"/>
 	<xacro:include filename="left_right.xacro"/>
+	<xacro:include filename="lr_limit.xacro"/>
 	<xacro:include filename="pelvis.xacro"/>
 	<xacro:include filename="leg.xacro"/>
@@ -16,4 +17,4 @@
 	<xacro:arm parent="torso" side="left"/>
 	<xacro:arm parent="torso" side="right"/>
-	<!--<xacro:head parent="torso"/>-->
+	<xacro:head parent="torso"/>
 </robot>

File: xacro/arm.xacro (robot description, xacro)
@@ -30,4 +30,5 @@
     		</inertial>
 	 	</link>
+	 	<!-- shoulder x (forward) -->
 	 	<joint name="shoulder_f_joint_${side}"
 	 		   type="revolute">
@@ -39,4 +40,5 @@
 	 		<limit lower="${-15*d2r}" upper="${90*d2r}" effort="10" velocity="10"/>
 	 	</joint>
+	 	<!-- shoulder y (side) -->
 	 	<joint name="shoulder_s_joint_${side}"
 	 		   type="revolute">
@@ -45,5 +47,5 @@
 	 		<origin xyz="0 0 0" rpy="0 0 0"/>
 	 		<axis xyz="0 1 0"/>
-	 		<limit lower="0" upper="${105*d2r}" effort="10" velocity="10"/>
+	 		<xacro:lr_limit side="${side}" lower="0" upper="${105*d2r}" effort="10" velocity="10"/>
 	 	</joint>
 	</xacro:macro>

File: xacro/head.xacro (robot description, xacro)
@@ -10,26 +10,82 @@
 		<link name="neck">
 	 		<xacro:meshes file="neck"/>
+	 		<inertial>
+	 			<origin xyz="0 -0.02 0.02" rpy="0 0 0"/>
+      			<mass value="0.633"/>
+      			<inertia ixx="1.0" ixy="1.0" ixz="1.0"
+      				     iyy="1.0" iyz="1.0"
+      				     izz="1.0"/>
+    		</inertial>
 	 	</link>
 	 	<link name="neck_fork">
 	 		<xacro:meshes file="neck_fork"/>
+	 		<inertial>
+	 			<!-- z unknown -->
+	 			<origin xyz="0.01 -0.01 -0.02" rpy="0 0 0"/>
+      			<mass value="0.444"/>
+      			<inertia ixx="1.0" ixy="1.0" ixz="1.0"
+      				     iyy="1.0" iyz="1.0"
+      				     izz="1.0"/>
+    		</inertial>
 	 	</link>
-	 	<joint name="neck_r_joint"
+	 	<link name="neck_cross">
+	 		<xacro:meshes file="neck_cross"/>
+	 		<inertial>
+	 			<origin xyz="-0.01 0.01 0" rpy="0 0 0"/>
+      			<mass value="0.320"/>
+      			<inertia ixx="1.0" ixy="1.0" ixz="1.0"
+      				     iyy="1.0" iyz="1.0"
+      				     izz="1.0"/>
+    		</inertial>
+	 	</link>
+	 	<link name="head">
+	 		<xacro:meshes file="head"/>
+	 		<inertial>
+	 			<origin xyz="0 0.04 0.06" rpy="0 0 0"/>
+      			<mass value="1.258"/>
+      			<inertia ixx="1.0" ixy="1.0" ixz="1.0"
+      				     iyy="1.0" iyz="1.0"
+      				     izz="1.0"/>
+    		</inertial>
+	 	</link>
+	 	<!-- neck x (forward) -->
+	 	<joint name="neck_f_joint"
 	 		   type="revolute">
 	 		<parent link="${parent}"/>
 	 		<child link="neck"/>
-	 		<!-- invalid Z -->
-	 		<origin xyz="0 0 0.145" rpy="0 0 0"/>
+	 		<!-- unknown -->
+	 		<origin xyz="0 0.041 0.016" rpy="0 0 0"/>
+	 		<axis xyz="-1 0 0"/>
+	 		<limit lower="${0*d2r}" upper="${60*d2r}" effort="10" velocity="10"/>
+	 	</joint>
+	 	<!-- head z (rotate) -->
+		<joint name="head_r_joint"
+			   type="revolute">
+			<parent link="neck"/>
+	 		<child link="neck_fork"/>
+	 		<!-- unknown -->
+	 		<origin xyz="0 -0.034 0.13" rpy="0 0 0"/>
 	 		<axis xyz="0 0 1"/>
 	 		<limit lower="${-90*d2r}" upper="${90*d2r}" effort="10" velocity="10"/>
-	 	</joint>
-	 	<joint name="neck_f_joint"
-	 		   type="revolute">
-	 		<parent link="neck"/>
-	 		<child link="neck_fork"/>
-	 		<!-- invalid Z -->
+		</joint>
+		<!-- head y (side) -->
+		<joint name="head_s_joint"
+			   type="revolute">
+			<parent link="neck_fork"/>
+	 		<child link="neck_cross"/>
+	 		<origin xyz="0 0 0" rpy="0 0 0"/>
+	 		<axis xyz="0 1 0"/>
+	 		<limit lower="${-15*d2r}" upper="${15*d2r}" effort="10" velocity="10"/>
+		</joint>
+		<!-- head x (forward) -->
+		<joint name="head_f_joint"
+			   type="revolute">
+			<parent link="neck_cross"/>
+	 		<child link="head"/>
+	 		<!-- z unknown -->
 	 		<origin xyz="0 0 0" rpy="0 0 0"/>
 	 		<axis xyz="1 0 0"/>
 	 		<limit lower="${-20*d2r}" upper="${30*d2r}" effort="10" velocity="10"/>
-	 	</joint>
+		</joint>
 	</xacro:macro>
 </robot>

File: xacro/left_right.xacro (robot description, xacro)
@@ -1,6 +1,6 @@
 <?xml version="1.0"?>
+<!-- Change Y-axis sign based on left/right side to allow mirror parts -->
 <robot xmlns:xacro="http://www.ros.org/wiki/xacro">
 	<xacro:macro name="left_right" params="side">
-		<!-- Change left/right x sign -->
 		<xacro:if value="${side == 'left'}">
   			<xacro:property scope="parent" name="x_sign" value="-1" />

File: xacro/leg.xacro (robot description, xacro)
@@ -86,5 +86,5 @@
 	 		<origin xyz="0 0 0" rpy="0 0 0"/>
 	 		<axis xyz="0 1 0"/>
-	 		<limit lower="${-11*d2r}" upper="${20*d2r}" effort="10" velocity="10"/>
+	 		<xacro:lr_limit side="${side}" lower="${-11*d2r}" upper="${20*d2r}" effort="10" velocity="10"/>
 	 	</joint>
 	 	<!-- hip x rotate (forward)-->
@@ -95,5 +95,5 @@
 	 		<origin xyz="0 0 0" rpy="0 0 0"/>
 	 		<axis xyz="1 0 0"/>
-	 		<limit lower="${-45*d2r}" upper="${70*d2r}" effort="10" velocity="10"/>
+	 		<limit lower="${-45*d2r}" upper="${70*d2r}" effort="10" velocity="10"/>-
 	 	</joint>
 	 	<!-- knee -->
@@ -122,5 +122,5 @@
 	 		<origin xyz="0 0 0" rpy="0 0 0"/>
 	 		<axis xyz="0 1 0"/>
-	 		<limit lower="${-20*d2r}" upper="${11*d2r}" effort="10" velocity="10"/>
+	 		<xacro:lr_limit side="${side}" lower="${-20*d2r}" upper="${11*d2r}" effort="10" velocity="10"/>
 	 	</joint>
  	</xacro:macro>

File: xacro/meshes.xacro (robot description, xacro)
@@ -1,3 +1,4 @@
 <?xml version="1.0"?>
+<!-- Create visual and collision with given mesh -->
 <robot xmlns:xacro="http://www.ros.org/wiki/xacro">
 	<xacro:macro name="meshes" params="file xyz:='0 0 0' rpy:='0 0 0'">
