Commit message: Fix inertia values from Inventor (fix axes and mass values). Fix transmission. Fix limits. Icrease efforts

File: xacro/ar600.xacro (robot description, xacro)
@@ -2,5 +2,4 @@
 <robot xmlns:xacro="http://www.ros.org/wiki/xacro" name="ar600">
 	<xacro:property name="d2r" value="0.01745329251994329577"/>
-	<xacro:property name="M_PI" value="3.14159"/>
 	<xacro:include filename="meshes.xacro"/>
 	<xacro:include filename="left_right.xacro"/>
@@ -9,19 +8,19 @@
 	<xacro:include filename="pelvis.xacro"/>
 	<xacro:include filename="leg.xacro"/>
-	<xacro:include filename="torso.xacro"/>
-	<xacro:include filename="arm.xacro"/>
-	<xacro:include filename="head.xacro"/>
+	<!-- <xacro:include filename="torso.xacro"/> -->
+	<!-- <xacro:include filename="arm.xacro"/> -->
+	<!-- <xacro:include filename="head.xacro"/> -->
 	<xacro:pelvis/>
+	<!-- Pelvis - base_link -->
 	<xacro:leg parent="base_link" side="left"/>
 	<xacro:leg parent="base_link" side="right"/>
-	<xacro:torso parent="base_link"/>
-	<xacro:arm parent="torso" side="left"/>
-	<xacro:arm parent="torso" side="right"/>
-	<xacro:head parent="torso"/>
-	<!-- ros_control plugin -->
-  	<!--<gazebo>
+	<!-- <xacro:torso parent="base_link"/> -->
+	<!-- <xacro:arm parent="torso" side="left"/> -->
+	<!-- <xacro:arm parent="torso" side="right"/> -->
+	<!-- <xacro:head parent="torso"/> -->
+  	<gazebo>
     	<plugin name="gazebo_ros_control" filename="libgazebo_ros_control.so">
-      	<robotNamespace>/ar600</robotNamespace>
+      	<!-- <robotNamespace>/ar600</robotNamespace> -->
     	</plugin>
-  	</gazebo>-->
+  	</gazebo>
 </robot>

File: xacro/arm.xacro (robot description, xacro)
@@ -38,5 +38,5 @@
 	 		<origin xyz="${0.197 * cos(10 * d2r) * x_sign} ${0.197 * sin(10 * d2r)} 0" rpy="0 0 ${10 * d2r * x_sign}"/>
 	 		<axis xyz="1 0 0"/>
-	 		<limit lower="${-15*d2r}" upper="${90*d2r}" effort="10" velocity="10"/>
+	 		<limit lower="${-15*d2r}" upper="${90*d2r}" effort="20" velocity="10"/>
 	 	</joint>
 	 	<!-- shoulder y (side) -->
@@ -47,5 +47,5 @@
 	 		<origin xyz="0 0 0" rpy="0 0 0"/>
 	 		<axis xyz="0 ${-x_sign} 0"/>
-	 		<xacro:lr_limit side="${side}" lower="0" upper="${105*d2r}" effort="10" velocity="10"/>
+	 		<xacro:lr_limit side="${side}" lower="0" upper="${105*d2r}" effort="20" velocity="10"/>
 	 	</joint>
 	 	<xacro:transmission_block joint_name="shoulder_f_joint_${side}"/>

File: xacro/leg.xacro (robot description, xacro)
@@ -14,8 +14,8 @@
 	 		<inertial>
 	 			<origin xyz="${-0.02 * x_sign} 0 0.07" rpy="0 0 0"/>
-      			<mass value="3.170"/>
-      			<inertia ixx="0.009316" ixy="-0.000234" ixz="0.002895"
-      				                    iyy="0.012979"  iyz="0.000000"
-      				                                    izz="0.006561"/>
+      			<mass value="0.907"/>
+      			<inertia ixx="0.004196" ixy="-0.000201" ixz="-0.000014"
+      				                    iyy="0.001524"  iyz="-0.000269"
+      				                                    izz="0.003769"/>
     		</inertial>
 	 	</link>
@@ -24,8 +24,8 @@
 	 		<inertial>
 	 			<origin xyz="${-0.03 * x_sign} 0.01 0.00" rpy="0 0 0"/>
-      			<mass value="1.799"/>
-      			<inertia ixx="0.001498" ixy="0.000126" ixz="0.000001"
-      				                    iyy="0.001990" iyz="-0.000016"
-      				                                   izz="0.002404"/>
+      			<mass value="0.754"/>
+      			<inertia ixx="0.001265" ixy="0.000000" ixz="0.000000"
+      				                    iyy="0.000786" iyz="0.000000"
+      				                                   izz="0.001560"/>
     		</inertial>
 	 	</link>
@@ -34,8 +34,11 @@
 	 		<inertial>
 	 			<origin xyz="${0.01 * x_sign} 0.00 -0.14" rpy="0 0 0"/>
-      			<mass value="6.779"/>
-      			<inertia ixx="0.037615" ixy="0.000139" ixz="-0.000896"
+      			<mass value="4.04"/>
+      			<!-- <inertia ixx="0.037615" ixy="0.000139" ixz="-0.000896"
       				                    iyy="0.031299" iyz="-0.000182"
-      				                                   izz="0.012270"/>
+      				                                   izz="0.012270"/> -->
+						<inertia ixx="0.035175" ixy="-0.000067" ixz="0.000877"
+      				                    iyy="0.040670" iyz="-0.000379"
+      				                                   izz="0.011745"/>
     		</inertial>
 	 	</link>
@@ -44,8 +47,11 @@
 	 		<inertial>
 	 			<origin xyz="0.00 0.01 -0.11" rpy="0 0 0"/>
-      			<mass value="1"/>
-      			<inertia ixx="0.028848" ixy="0.000053" ixz="-0.000056"
+      			<mass value="2.24"/>
+      			<!-- <inertia ixx="0.028848" ixy="0.000053" ixz="-0.000056"
       				                    iyy="0.026849" iyz="0.001709"
-      				                                   izz="0.005196"/>
+      				                                   izz="0.005196"/> -->
+						<inertia ixx="0.011381" ixy="0.000079" ixz="0.000000"
+      				                    iyy="0.013862" iyz="-0.000663"
+      				                                   izz="0.005662"/>
     		</inertial>
 	 	</link>
@@ -54,8 +60,8 @@
 	 		<inertial>
 	 			<origin xyz="${-0.02 * x_sign} 0.01 0.00" rpy="0 0 0"/>
-      			<mass value="1"/>
-      			<inertia ixx="0.000424" ixy="-0.000001" ixz="-0.000001"
-      				                    iyy="0.000603"  iyz="0.000001"
-      				                                    izz="0.000898"/>
+      			<mass value="0.297"/>
+      			<inertia ixx="0.000283" ixy="0.000000" ixz="0.000000"
+      				                    iyy="0.000161"  iyz="0.000000"
+      				                                    izz="0.000346"/>
     		</inertial>
 	 	</link>
@@ -64,8 +70,11 @@
 	 		<inertial>
 	 			<origin xyz="${0.03 * x_sign} 0.00 -0.06" rpy="0 0 0"/>
-      			<mass value="1"/>
-      			<inertia ixx="0.006101" ixy="-0.000307" ixz="-0.001261"
+      			<mass value="2.2"/>
+      			<!-- <inertia ixx="0.006101" ixy="-0.000307" ixz="-0.001261"
       				                    iyy="0.012336"  iyz="0.000060"
-      				                                    izz="0.013546"/>
+      				                                    izz="0.013546"/> -->
+						<inertia ixx="0.013004" ixy="-0.000212" ixz="0.000096"
+      															iyy="0.005467" iyz="0.001058"
+      				                                  		izz="0.015293"/>
     		</inertial>
 	 	</link>
@@ -77,5 +86,6 @@
 	 		<origin xyz="${0.088 * x_sign} 0.0276 0" rpy="0 0 0"/>
 	 		<axis xyz="0 0 ${-x_sign}"/>
-	 		<limit lower="${-20*d2r}" upper="${20*d2r}" effort="10" velocity="10"/>
+	 		<limit lower="${-20*d2r}" upper="${20*d2r}" effort="100" velocity="10"/>
+			 <dynamics damping="0.1" friction="0.0"/>
 	 	</joint>
 	 	<!-- hip y rotate (side)-->
@@ -86,5 +96,6 @@
 	 		<origin xyz="0 0 0" rpy="0 0 0"/>
 	 		<axis xyz="0 ${-x_sign} 0"/>
-	 		<xacro:lr_limit side="${side}" lower="${-11*d2r}" upper="${20*d2r}" effort="10" velocity="10"/>
+	 		<xacro:lr_limit side="${side}" lower="${-11*d2r}" upper="${20*d2r}" effort="1000" velocity="10"/>
+			 <dynamics damping="0.1" friction="0.0"/>
 	 	</joint>
 	 	<!-- hip x rotate (forward)-->
@@ -95,5 +106,6 @@
 	 		<origin xyz="0 0 0" rpy="0 0 0"/>
 	 		<axis xyz="1 0 0"/>
-	 		<limit lower="${-45*d2r}" upper="${70*d2r}" effort="10" velocity="10"/>-
+	 		<limit lower="${-45*d2r}" upper="${70*d2r}" effort="100" velocity="10"/>
+			<dynamics damping="0.1" friction="0.0"/>
 	 	</joint>
 	 	<!-- knee -->
@@ -104,5 +116,6 @@
 	 		<origin xyz="0 0 -0.28" rpy="0 0 0"/>
 	 		<axis xyz="1 0 0"/>
-	 		<limit lower="${-140*d2r}" upper="0" effort="10" velocity="10"/>
+	 		<limit lower="${-140*d2r}" upper="0" effort="100" velocity="10"/>
+			 <dynamics damping="0.1" friction="0.0"/>
 	 	</joint>
 	 	<!-- ankle x (forward) -->
@@ -113,5 +126,6 @@
 	 		<origin xyz="0 0 -0.28" rpy="0 0 0"/>
 	 		<axis xyz="1 0 0"/>
-	 		<limit lower="${-33*d2r}" upper="${70*d2r}" effort="10" velocity="10"/>
+	 		<limit lower="${-33*d2r}" upper="${70*d2r}" effort="100" velocity="10"/>
+			 <dynamics damping="0.1" friction="0.0"/>
 	 	</joint>
 	 	<!-- ankle y (side) -->
@@ -122,5 +136,6 @@
 	 		<origin xyz="0 0 0" rpy="0 0 0"/>
 	 		<axis xyz="0 ${-x_sign} 0"/>
-	 		<xacro:lr_limit side="${side}" lower="${-20*d2r}" upper="${11*d2r}" effort="10" velocity="10"/>
+	 		<xacro:lr_limit side="${side}" lower="${-20*d2r}" upper="${11*d2r}" effort="100" velocity="10"/>
+			<dynamics damping="0.1" friction="0.0"/>
 	 	</joint>
 	 	<xacro:transmission_block joint_name="hip_r_joint_${side}"/>

File: xacro/lr_limit.xacro (robot description, xacro)
@@ -3,10 +3,10 @@
 <robot xmlns:xacro="http://www.ros.org/wiki/xacro">
 	<xacro:macro name="lr_limit" params="side lower upper effort velocity">
-		<xacro:if value="${side == 'left'}">
+		<!-- <xacro:if value="${side == 'left'}"> -->
   			<limit lower="${lower}" upper="${upper}" effort="${effort}" velocity="${velocity}"/>
-		</xacro:if>
-		<xacro:if value="${side == 'right'}">
+		<!-- </xacro:if> -->
+		<!-- <xacro:if value="${side == 'right'}">
   			<limit lower="${-upper}" upper="${-lower}" effort="${effort}" velocity="${velocity}"/>
-		</xacro:if>
+		</xacro:if>	 -->
  	</xacro:macro>
 </robot>

File: xacro/pelvis.xacro (robot description, xacro)
@@ -14,8 +14,8 @@
 	 			<!-- z origin is incorrect -->
 	 			<origin xyz="0 0 0.15" rpy="0 0 0"/>
-      			<mass value="5.045"/>
-      			<inertia ixx="0.031053" ixy="0.000014" ixz="-0.000227"
-      				                    iyy="0.012429" iyz="-0.000016"
-      				                                   izz="0.032811"/>
+      			<mass value="4.127"/>
+      			<inertia ixx="0.011960" ixy="-0.000003" ixz="0.000002"
+      				                    iyy="0.028330" iyz="0.000108"
+      				                                   izz="0.033849"/>
     		</inertial>
 	 	</link>

File: xacro/torso.xacro (robot description, xacro)
@@ -13,6 +13,5 @@
     		</inertial>
 	 	</link>
-	 	<joint name="torso_r_joint"
-	 		   type="revolute">
+	 	<joint name="torso_r_joint" type="revolute">
 	 		<parent link="${parent}"/>
 	 		<child link="torso"/>
@@ -20,5 +19,5 @@
 	 		<origin xyz="0 0 0.46" rpy="0 0 0"/>
 	 		<axis xyz="0 0 1"/>
-	 		<limit lower="${-45*d2r}" upper="${45*d2r}" effort="10" velocity="10"/>
+	 		<limit lower="${-45*d2r}" upper="${45*d2r}" effort="50" velocity="10"/>
 	 	</joint>
 	 	<xacro:transmission_block joint_name="torso_r_joint"/>

File: xacro/transmission_block.xacro (robot description, xacro)
@@ -5,8 +5,10 @@
       	<type>transmission_interface/SimpleTransmission</type>
       	<joint name="${joint_name}">
-        		<hardwareInterface>hardware_interface/PositionJointInterface</hardwareInterface>
+        		<!-- <hardwareInterface>hardware_interface/PositionJointInterface</hardwareInterface> -->
+				<hardwareInterface>hardware_interface/EffortJointInterface</hardwareInterface>
       	</joint>
       	<actuator name="${joint_name}_motor">
-        		<hardwareInterface>hardware_interface/PositionJointInterface</hardwareInterface>
+        		<!-- <hardwareInterface>hardware_interface/PositionJointInterface</hardwareInterface> -->
+				<hardwareInterface>hardware_interface/EffortJointInterface</hardwareInterface>
         		<mechanicalReduction>1</mechanicalReduction>
       	</actuator>

Commit message: Fix URDF and add RVIZ config

File: xacro/ar600.xacro (robot description, xacro)
@@ -8,7 +8,7 @@
 	<xacro:include filename="pelvis.xacro"/>
 	<xacro:include filename="leg.xacro"/>
-	<!-- <xacro:include filename="torso.xacro"/> -->
+	<xacro:include filename="torso.xacro"/>
 	<!-- <xacro:include filename="arm.xacro"/> -->
-	<!-- <xacro:include filename="head.xacro"/> -->
+	<xacro:include filename="head_and_neck.xacro"/>
 	<xacro:pelvis/>
 	<!-- Pelvis - base_link -->
@@ -18,5 +18,5 @@
 	<!-- <xacro:arm parent="torso" side="left"/> -->
 	<!-- <xacro:arm parent="torso" side="right"/> -->
-	<!-- <xacro:head parent="torso"/> -->
+	<!-- <xacro:head_and_neck parent="torso"/> -->
   	<gazebo>
     	<plugin name="gazebo_ros_control" filename="libgazebo_ros_control.so">

File: xacro/head_and_neck.xacro (robot description, xacro)
@@ -7,13 +7,13 @@
 		z <-  y
 	-->
-	<xacro:macro name="head" params="parent">
+	<xacro:macro name="head_and_neck" params="parent">
 		<link name="neck">
 	 		<xacro:meshes file="neck"/>
 	 		<inertial>
-	 			<origin xyz="-0.02 0.00 0.02" rpy="0 0 0"/>
-      			<mass value="0.633"/>
-      			<inertia ixx="0.000884" ixy="0.000001" ixz="-0.000246"
-      				                    iyy="0.000982" iyz="0.000500"
-      				                                   izz="0.000627"/>
+	 			<origin xyz="-0.00 0.00 0.02" rpy="0 0 0"/>
+      	<mass value="0.657"/>
+      	<inertia ixx="0.001201" ixy="0.000000" ixz="-0.000000"
+      				                  iyy="0.001020" iyz="0.000300"
+      				                                 izz="0.000718"/>
     		</inertial>
 	 	</link>
@@ -22,9 +22,9 @@
 	 		<inertial>
 	 			<!-- z unknown -->
-	 			<origin xyz="0.01 -0.01 -0.02" rpy="0 0 0"/>
-      			<mass value="0.444"/>
-      			<inertia ixx="0.000285" ixy="-0.000016" ixz="0.000073"
-      				                    iyy="0.000401"  iyz="-0.000021"
-      				                                    izz="0.000238"/>
+	 			<origin xyz="0 -0.01 -0.02" rpy="0 0 0"/>
+      	<mass value="0.016"/>
+      	<inertia ixx="0.000013" ixy="-0.000000" ixz="0.000000"
+      				                  iyy="0.000006"  iyz="0.000000"
+      				                                  izz="0.000012"/>
     		</inertial>
 	 	</link>
@@ -32,20 +32,20 @@
 	 		<xacro:meshes file="neck_cross"/>
 	 		<inertial>
-	 			<origin xyz="0.01 0.01 0" rpy="0 0 0"/>
-      			<mass value="0.320"/>
-      			<inertia ixx="0.000054" ixy="-0.000002" ixz="0.000000"
-      				                    iyy="0.000054"  iyz="0.000000"
-      				                                    izz="0.000092"/>
+	 			<origin xyz="0 0 0" rpy="0 0 0"/>
+      	<mass value="0.140"/>
+      	<inertia ixx="0.000026" ixy="0.000000" ixz="0.000000"
+      				                  iyy="0.000256" iyz="0.000000"
+      				                                 izz="0.000266"/>
     		</inertial>
 	 	</link>
 	 	<link name="head">
-	 		<xacro:meshes file="head" collision="True"/>
+	 		<xacro:meshes file="head"/>
 	 		<inertial>
-	 			<origin xyz="0.04 0.00 0.06" rpy="0 0 0"/>
-      			<mass value="1.258"/>
-      			<inertia ixx="0.005118" ixy="-0.000058" ixz="-0.000120"
-      				                    iyy="0.005112"  iyz="-0.000172"
-      				                                    izz="0.005643"/>
-    		</inertial>
+	 			<origin xyz="0.00 0.00 0.06" rpy="0 0 0"/>
+      		<mass value="5.515"/>
+      		<inertia ixx="0.033638" ixy="0.000000" ixz="0.000001"
+      				                    iyy="0.031846"  iyz="0.002895"
+      				                                    izz="0.138931"/>
+    	</inertial>
 	 	</link>
 	 	<!-- neck x (forward) -->

File: xacro/leg.xacro (robot description, xacro)
@@ -15,5 +15,5 @@
 	 			<origin xyz="${-0.02 * x_sign} 0 0.07" rpy="0 0 0"/>
       			<mass value="0.907"/>
-      			<inertia ixx="0.004196" ixy="-0.000201" ixz="-0.000014"
+      			<inertia ixx="0.004196" ixy="${-x_sign * 0.000201}" ixz="${-x_sign * 0.000014}"
       				                    iyy="0.001524"  iyz="-0.000269"
       				                                    izz="0.003769"/>
@@ -35,7 +35,4 @@
 	 			<origin xyz="${0.01 * x_sign} 0.00 -0.14" rpy="0 0 0"/>
       			<mass value="4.04"/>
-      			<!-- <inertia ixx="0.037615" ixy="0.000139" ixz="-0.000896"
-      				                    iyy="0.031299" iyz="-0.000182"
-      				                                   izz="0.012270"/> -->
 						<inertia ixx="0.035175" ixy="-0.000067" ixz="0.000877"
       				                    iyy="0.040670" iyz="-0.000379"
@@ -48,7 +45,4 @@
 	 			<origin xyz="0.00 0.01 -0.11" rpy="0 0 0"/>
       			<mass value="2.24"/>
-      			<!-- <inertia ixx="0.028848" ixy="0.000053" ixz="-0.000056"
-      				                    iyy="0.026849" iyz="0.001709"
-      				                                   izz="0.005196"/> -->
 						<inertia ixx="0.011381" ixy="0.000079" ixz="0.000000"
       				                    iyy="0.013862" iyz="-0.000663"
@@ -71,7 +65,4 @@
 	 			<origin xyz="${0.03 * x_sign} 0.00 -0.06" rpy="0 0 0"/>
       			<mass value="2.2"/>
-      			<!-- <inertia ixx="0.006101" ixy="-0.000307" ixz="-0.001261"
-      				                    iyy="0.012336"  iyz="0.000060"
-      				                                    izz="0.013546"/> -->
 						<inertia ixx="0.013004" ixy="-0.000212" ixz="0.000096"
       															iyy="0.005467" iyz="0.001058"
@@ -79,4 +70,13 @@
     		</inertial>
 	 	</link>
+		<gazebo reference="foot_${side}">
+			<kp>100000.0</kp>
+			<kd>100.0</kd>
+			<mu1>0.9</mu1>
+			<mu2>0.09</mu2>
+			<fdir1>1 1 0</fdir1>
+			<maxVel>1.0</maxVel>
+			<minDepth>0.0001</minDepth>
+		</gazebo>
 	 	<!-- hip z rotate (vertical)-->
 	 	<joint name="hip_r_joint_${side}"
@@ -86,5 +86,5 @@
 	 		<origin xyz="${0.088 * x_sign} 0.0276 0" rpy="0 0 0"/>
 	 		<axis xyz="0 0 ${-x_sign}"/>
-	 		<limit lower="${-20*d2r}" upper="${20*d2r}" effort="100" velocity="10"/>
+	 		<limit lower="${-20*d2r}" upper="${20*d2r}" effort="1000" velocity="10"/>
 			 <dynamics damping="0.1" friction="0.0"/>
 	 	</joint>
@@ -96,5 +96,5 @@
 	 		<origin xyz="0 0 0" rpy="0 0 0"/>
 	 		<axis xyz="0 ${-x_sign} 0"/>
-	 		<xacro:lr_limit side="${side}" lower="${-11*d2r}" upper="${20*d2r}" effort="1000" velocity="10"/>
+	 		<xacro:lr_limit side="${side}" lower="${-25*d2r}" upper="${25*d2r}" effort="1000" velocity="10"/>
 			 <dynamics damping="0.1" friction="0.0"/>
 	 	</joint>
@@ -104,7 +104,7 @@
 	 		<parent link="hip_cross_${side}"/>
 	 		<child link="hip_${side}"/>
-	 		<origin xyz="0 0 0" rpy="0 0 0"/>
+	 		<origin xyz="0 0 0" rpy="${ 0 * d2r} 0 0"/>
 	 		<axis xyz="1 0 0"/>
-	 		<limit lower="${-45*d2r}" upper="${70*d2r}" effort="100" velocity="10"/>
+	 		<limit lower="${-45*d2r}" upper="${70*d2r}" effort="1000" velocity="10"/>
 			<dynamics damping="0.1" friction="0.0"/>
 	 	</joint>
@@ -116,5 +116,5 @@
 	 		<origin xyz="0 0 -0.28" rpy="0 0 0"/>
 	 		<axis xyz="1 0 0"/>
-	 		<limit lower="${-140*d2r}" upper="0" effort="100" velocity="10"/>
+	 		<limit lower="${-140*d2r}" upper="0" effort="1000" velocity="10"/>
 			 <dynamics damping="0.1" friction="0.0"/>
 	 	</joint>
@@ -126,5 +126,5 @@
 	 		<origin xyz="0 0 -0.28" rpy="0 0 0"/>
 	 		<axis xyz="1 0 0"/>
-	 		<limit lower="${-33*d2r}" upper="${70*d2r}" effort="100" velocity="10"/>
+	 		<limit lower="${-70*d2r}" upper="${70*d2r}" effort="1000" velocity="10"/>
 			 <dynamics damping="0.1" friction="0.0"/>
 	 	</joint>
@@ -136,5 +136,5 @@
 	 		<origin xyz="0 0 0" rpy="0 0 0"/>
 	 		<axis xyz="0 ${-x_sign} 0"/>
-	 		<xacro:lr_limit side="${side}" lower="${-20*d2r}" upper="${11*d2r}" effort="100" velocity="10"/>
+	 		<xacro:lr_limit side="${side}" lower="${-25*d2r}" upper="${25*d2r}" effort="1000" velocity="10"/>
 			<dynamics damping="0.1" friction="0.0"/>
 	 	</joint>

File: xacro/torso.xacro (robot description, xacro)
@@ -7,8 +7,8 @@
 	 			<!-- origin is incorrect -->
 	 			<origin xyz="0 0 -0.09" rpy="0 0 0"/>
-      			<mass value="29.642"/>
-      			<inertia ixx="0.118418" ixy="-0.000174" ixz="0.001227"
-      				                    iyy="0.091310"  iyz="-0.000488"
-      				                                    izz="0.061124"/>
+      			<mass value="13.420"/>
+      			<inertia ixx="0.141741" ixy="0.000000" ixz="0.000001"
+      				                    iyy="0.178527"  iyz="0.003353"
+      				                                    izz="0.107042"/>
     		</inertial>
 	 	</link>
